File: template/GameBoy_GamePak_AGB-002_Bootleg/GameBoy_GamePak_AGB-002_Bootleg.kicad_pcb (KiCad board)
At the start: 2 copper layers, 52.3 x 32 mm, 1 part, among them J1 GameBoy_GamePak_AGB-002

Commit message: Update all files to KiCAD 6.x format
Other:
- net class Default removed
