File: template/GameBoy_GamePak_DMG-09_Bootleg_UltraShort/GameBoy_GamePak_DMG-09_Bootleg_UltraShort.kicad_pcb (KiCad board)
At the start: 2 copper layers, 53 x 28.4 mm, 1 part, among them J1 GameBoy_GamePak_DMG-09

Commit message: Update all files to KiCAD 6.x format
Other:
- net class Default removed
